Commit message: part 2 of e done

File: body.urdf (robot description, URDF)
Before this commit: robot robot, 5 links, 4 joints
Links:
- removed link Link3
- removed link Link4
Joints:
- removed joint Link1_Link2
- removed joint Link2_Link3
- removed joint Link3_Link4
- added joint Link0_Link2: type revolute, parent Link0, child Link2, origin xyz=0.5 1.5 1 rpy=0 0 0, axis 0 1 0, limit lower=-3.14159 upper=3.14159 effort=0.0 velocity=0.0
- joint Link0_Link1: origin xyz=0 0 1 rpy=0 0 0 -> xyz=0.5 0.5 1 rpy=0 0 0

Commit message: sensors

File: body.urdf (robot description, URDF)
Before this commit: robot robot, 3 links, 2 joints
Joints:
- joint Link0_Link1: origin xyz=0.5 0.5 1 rpy=0 0 0 -> xyz=0 0.5 1 rpy=0 0 0
- joint Link0_Link2: origin xyz=0.5 1.5 1 rpy=0 0 0 -> xyz=0 1.5 1 rpy=0 0 0

Commit message: upto Random Movement

File: body.urdf (robot description, URDF)
Before this commit: robot robot, 3 links, 2 joints
Joints:
- joint Link0_Link1: origin xyz=0 0.5 1 rpy=0 0 0 -> xyz=1 0 2 rpy=0 0 0
- joint Link0_Link2: origin xyz=0 1.5 1 rpy=0 0 0 -> xyz=2 0 2 rpy=0 0 0

Commit message: k

File: body.urdf (robot description, URDF)
Before this commit: robot robot, 3 links, 2 joints
Joints:
- joint Link0_Link1: origin xyz=1 0 2 rpy=0 0 0 -> xyz=0.5 0 1 rpy=0 0 0
- joint Link0_Link2: origin xyz=2 0 2 rpy=0 0 0 -> xyz=-0.5 0 1 rpy=0 0 0

Commit message: N

File: body.urdf (robot description, URDF)
Before this commit: robot robot, 3 links, 2 joints
Links:
- removed link Link0
- removed link Link1
- removed link Link2
- added link BackLeg, mass 1; collision box size=0.2 1 0.2; visual box size=0.2 1 0.2
- added link FrontLeg, mass 1; collision box size=0.2 1 0.2; visual box size=0.2 1 0.2
- added link LeftLeg, mass 1; collision box size=1 0.2 0.2; visual box size=1 0.2 0.2
- added link LowerBackLeg, mass 1; collision box size=0.2 0.2 1; visual box size=0.2 0.2 1
- added link LowerFrontLeg, mass 1; collision box size=0.2 0.2 1; visual box size=0.2 0.2 1
- added link LowerLeftLeg, mass 1; collision box size=0.2 0.2 1; visual box size=0.2 0.2 1
- added link LowerRightLeg, mass 1; collision box size=0.2 0.2 1; visual box size=0.2 0.2 1
- added link RightLeg, mass 1; collision box size=1 0.2 0.2; visual box size=1 0.2 0.2
- added link Torso, mass 1; collision box size=1 1 0.5; visual box size=1 1 0.5
Joints:
- removed joint Link0_Link1
- removed joint Link0_Link2
- added joint BackLeg_LowerBackLeg: type revolute, parent BackLeg, child LowerBackLeg, origin xyz=0 -1 0 rpy=0 0 0, axis 0 1 0, limit lower=-3.14159 upper=3.14159 effort=0.0 velocity=0.0
- added joint FrontLeg_LowerFrontLeg: type revolute, parent FrontLeg, child LowerFrontLeg, origin xyz=0 1 0 rpy=0 0 0, axis 0 1 0, limit lower=-3.14159 upper=3.14159 effort=0.0 velocity=0.0
- added joint LeftLeg_LowerLeftLeg: type revolute, parent LeftLeg, child LowerLeftLeg, origin xyz=-1 0 0 rpy=0 0 0, axis 1 0 0, limit lower=-3.14159 upper=3.14159 effort=0.0 velocity=0.0
- added joint RightLeg_LowerRightLeg: type revolute, parent RightLeg, child LowerRightLeg, origin xyz=1 0 0 rpy=0 0 0, axis 1 0 0, limit lower=-3.14159 upper=3.14159 effort=0.0 velocity=0.0
- added joint Torso_BackLeg: type revolute, parent Torso, child BackLeg, origin xyz=0 -0.5 1 rpy=0 0 0, axis 1 0 0, limit lower=-3.14159 upper=3.14159 effort=0.0 velocity=0.0
- added joint Torso_FrontLeg: type revolute, parent Torso, child FrontLeg, origin xyz=0 0.5 1 rpy=0 0 0, axis 1 0 0, limit lower=-3.14159 upper=3.14159 effort=0.0 velocity=0.0
- added joint Torso_LeftLeg: type revolute, parent Torso, child LeftLeg, origin xyz=-0.5 0 1 rpy=0 0 0, axis 0 1 0, limit lower=-3.14159 upper=3.14159 effort=0.0 velocity=0.0
- added joint Torso_RightLeg: type revolute, parent Torso, child RightLeg, origin xyz=0.5 0 1 rpy=0 0 0, axis 0 1 0, limit lower=-3.14159 upper=3.14159 effort=0.0 velocity=0.0

Commit message: assign 5

File: body.urdf (robot description, URDF)
Before this commit: robot robot, 9 links, 8 joints
Links:
- added link BLLowerLeg, mass 1; collision box size=[0.22589865] [0.25235909] [1.04276911]; visual box size=[0.22589865] [0.25235909] [1.04276911]
- added link BRLowerLeg, mass 1; collision box size=[0.22589865] [0.25235909] [1.04276911]; visual box size=[0.22589865] [0.25235909] [1.04276911]
- added link FLLowerLeg, mass 1; collision box size=[0.22589865] [0.25235909] [1.04276911]; visual box size=[0.22589865] [0.25235909] [1.04276911]
- added link FRLowerLeg, mass 1; collision box size=[0.22589865] [0.25235909] [1.04276911]; visual box size=[0.22589865] [0.25235909] [1.04276911]
Joints:
- added joint Torso_BLLowerLeg: type revolute, parent Torso, child BLLowerLeg, origin xyz=-0.5 -0.5 1 rpy=0 0 0, axis 0 0 1, limit lower=-3.14159 upper=3.14159 effort=0.0 velocity=0.0
- added joint Torso_BRLowerLeg: type revolute, parent Torso, child BRLowerLeg, origin xyz=0.5 -0.5 1 rpy=0 0 0, axis 1 0 0, limit lower=-3.14159 upper=3.14159 effort=0.0 velocity=0.0
- added joint Torso_FLLowerLeg: type revolute, parent Torso, child FLLowerLeg, origin xyz=-0.5 0.5 1 rpy=0 0 0, axis 0 1 1, limit lower=-3.14159 upper=3.14159 effort=0.0 velocity=0.0
- added joint Torso_FRLowerLeg: type revolute, parent Torso, child FRLowerLeg, origin xyz=0.5 0.5 1 rpy=0 0 0, axis 1 1 0, limit lower=-3.14159 upper=3.14159 effort=0.0 velocity=0.0

Commit message: readme updated

File: body.urdf (robot description, URDF)
Before this commit: robot robot, 13 links, 12 joints
Links:
- link BLLowerLeg: geometry collision box size=0.2 0.2 1; visual box size=0.2 0.2 1
- link BRLowerLeg: geometry collision box size=0.2 0.2 1; visual box size=0.2 0.2 1
- link FLLowerLeg: geometry collision box size=0.2 0.2 1; visual box size=0.2 0.2 1
- link FRLowerLeg: geometry collision box size=0.2 0.2 1; visual box size=0.2 0.2 1

Commit message: clean

File: body.urdf (robot description, URDF)
Before this commit: robot robot, 13 links, 12 joints
Links:
- link BLLowerLeg: geometry collision box size=[0.36876678] [0.22447758] [1.1385834]; visual box size=[0.36876678] [0.22447758] [1.1385834]
- link BRLowerLeg: geometry collision box size=[0.36876678] [0.22447758] [1.1385834]; visual box size=[0.36876678] [0.22447758] [1.1385834]
- link FLLowerLeg: geometry collision box size=[0.36876678] [0.22447758] [1.1385834]; visual box size=[0.36876678] [0.22447758] [1.1385834]
- link FRLowerLeg: geometry collision box size=[0.36876678] [0.22447758] [1.1385834]; visual box size=[0.36876678] [0.22447758] [1.1385834]

Commit message: debugging

File: body.urdf (robot description, URDF)
Before this commit: robot robot, 13 links, 12 joints
Links:
- removed link BLLowerLeg
- removed link BRLowerLeg
- removed link BackLeg
- removed link FLLowerLeg
- removed link FRLowerLeg
- removed link FrontLeg
- removed link LeftLeg
- removed link LowerBackLeg
- removed link LowerFrontLeg
- removed link LowerLeftLeg
- removed link LowerRightLeg
- removed link RightLeg
- removed link Torso
- added link Link0, mass 1; collision box size=0.08991598044376614 0.9442748055252959 0.3382065084119751; visual box size=0.08991598044376614 0.9442748055252959 0.3382065084119751
- added link Link1, mass 1; collision box size=0.0455999221821779 0.02686977156738546 0.6697390433067876; visual box size=0.0455999221821779 0.02686977156738546 0.6697390433067876
- added link Link2, mass 1; collision box size=0.09512630658809684 0.16538848030978914 0.34434555972075376; visual box size=0.09512630658809684 0.16538848030978914 0.34434555972075376
- added link Link3, mass 1; collision box size=0.8988646662309098 0.9302012553151247 0.7396883322632737; visual box size=0.8988646662309098 0.9302012553151247 0.7396883322632737
- added link Link4, mass 1; collision box size=0.6022585213627594 0.3154890842021959 0.7539458440226775; visual box size=0.6022585213627594 0.3154890842021959 0.7539458440226775
- added link Link5, mass 1; collision box size=0.2471946032366631 0.200022151378765 0.697997747025809; visual box size=0.2471946032366631 0.200022151378765 0.697997747025809
- added link Link6, mass 1; collision box size=0.5166362385928098 0.478293854473812 0.4242463320739529; visual box size=0.5166362385928098 0.478293854473812 0.4242463320739529
- added link Link7, mass 1; collision box size=0.49852502806705734 0.7303765293347746 0.895738399873903; visual box size=0.49852502806705734 0.7303765293347746 0.895738399873903
- added link Link8, mass 1; collision box size=0.7256492995698836 0.5686717320517842 0.5397813135865623; visual box size=0.7256492995698836 0.5686717320517842 0.5397813135865623
- added link Link9, mass 1; collision box size=0.5927177378189967 0.1787183874348065 0.21808294324593447; visual box size=0.5927177378189967 0.1787183874348065 0.21808294324593447
Joints:
- removed joint BackLeg_LowerBackLeg
- removed joint FrontLeg_LowerFrontLeg
- removed joint LeftLeg_LowerLeftLeg
- removed joint RightLeg_LowerRightLeg
- removed joint Torso_BLLowerLeg
- removed joint Torso_BRLowerLeg
- removed joint Torso_BackLeg
- removed joint Torso_FLLowerLeg
- removed joint Torso_FRLowerLeg
- removed joint Torso_FrontLeg
- removed joint Torso_LeftLeg
- removed joint Torso_RightLeg
- added joint Link0_Link1: type revolute, parent Link0, child Link1, origin xyz=0 0.47213740276264793 0.3382065084119751 rpy=0 0 0, axis 1 0 0, limit lower=-3.14159 upper=3.14159 effort=0.0 velocity=0.0
- added joint Link1_Link2: type revolute, parent Link1, child Link2, origin xyz=0 0.0455999221821779 0.6697390433067876 rpy=0 0 0, axis 1 0 0, limit lower=-3.14159 upper=3.14159 effort=0.0 velocity=0.0
- added joint Link2_Link3: type revolute, parent Link2, child Link3, origin xyz=0 0.09512630658809684 0.34434555972075376 rpy=0 0 0, axis 1 0 0, limit lower=-3.14159 upper=3.14159 effort=0.0 velocity=0.0
- added joint Link3_Link4: type revolute, parent Link3, child Link4, origin xyz=0 0.8988646662309098 0.7396883322632737 rpy=0 0 0, axis 1 0 0, limit lower=-3.14159 upper=3.14159 effort=0.0 velocity=0.0
- added joint Link4_Link5: type revolute, parent Link4, child Link5, origin xyz=0 0.6022585213627594 0.7539458440226775 rpy=0 0 0, axis 1 0 0, limit lower=-3.14159 upper=3.14159 effort=0.0 velocity=0.0
- added joint Link5_Link6: type revolute, parent Link5, child Link6, origin xyz=0 0.2471946032366631 0.697997747025809 rpy=0 0 0, axis 1 0 0, limit lower=-3.14159 upper=3.14159 effort=0.0 velocity=0.0
- added joint Link6_Link7: type revolute, parent Link6, child Link7, origin xyz=0 0.5166362385928098 0.4242463320739529 rpy=0 0 0, axis 1 0 0, limit lower=-3.14159 upper=3.14159 effort=0.0 velocity=0.0
- added joint Link7_Link8: type revolute, parent Link7, child Link8, origin xyz=0 0.49852502806705734 0.895738399873903 rpy=0 0 0, axis 1 0 0, limit lower=-3.14159 upper=3.14159 effort=0.0 velocity=0.0
- added joint Link8_Link9: type revolute, parent Link8, child Link9, origin xyz=0 0.7256492995698836 0.5397813135865623 rpy=0 0 0, axis 1 0 0, limit lower=-3.14159 upper=3.14159 effort=0.0 velocity=0.0
- added joint Link9_Link10: type revolute, parent Link9, child Link10, origin xyz=0 0.5927177378189967 0.21808294324593447 rpy=0 0 0, axis 1 0 0, limit lower=-3.14159 upper=3.14159 effort=0.0 velocity=0.0

Commit message: minor hcange

File: body.urdf (robot description, URDF)
Before this commit: robot robot, 10 links, 10 joints
Links:
- link Link0: geometry collision box size=0.7529831723212046 0.565117007555887 0.8030191664109855; visual box size=0.7529831723212046 0.565117007555887 0.8030191664109855
- link Link1: geometry collision box size=0.19415024083530874 0.14254383338228904 0.936509516854282; visual box size=0.19415024083530874 0.14254383338228904 0.936509516854282
- link Link2: geometry collision box size=0.48820175054702664 0.6794152478660177 0.8281490012226346; visual box size=0.48820175054702664 0.6794152478660177 0.8281490012226346
- link Link3: geometry collision box size=0.233756348616039 0.8891640217555714 0.07162717173401223; visual box size=0.233756348616039 0.8891640217555714 0.07162717173401223
- link Link4: geometry collision box size=0.7114452413300312 0.7483867602724774 0.6620237559790881; visual box size=0.7114452413300312 0.7483867602724774 0.6620237559790881
- link Link5: geometry collision box size=0.4849924955659737 0.6248998883589717 0.1457264134121834; visual box size=0.4849924955659737 0.6248998883589717 0.1457264134121834
- link Link6: geometry collision box size=0.8234380003730708 0.6041393145370686 0.953817394295689; visual box size=0.8234380003730708 0.6041393145370686 0.953817394295689
- link Link7: geometry collision box size=0.76079497129132 0.3726822485112079 0.186407095701565; visual box size=0.76079497129132 0.3726822485112079 0.186407095701565
- link Link8: geometry collision box size=0.9055970329906969 0.7540676214162395 0.8884605437782; visual box size=0.9055970329906969 0.7540676214162395 0.8884605437782
- link Link9: geometry collision box size=0.5195126159055607 0.8137197244535254 0.38693715368187753; visual box size=0.5195126159055607 0.8137197244535254 0.38693715368187753
Joints:
- joint Link0_Link1: origin xyz=0 0.47213740276264793 0.3382065084119751 rpy=0 0 0 -> xyz=0 0.2825585037779435 0.8030191664109855 rpy=0 0 0
- joint Link1_Link2: origin xyz=0 0.0455999221821779 0.6697390433067876 rpy=0 0 0 -> xyz=0 0.19415024083530874 0.936509516854282 rpy=0 0 0
- joint Link2_Link3: origin xyz=0 0.09512630658809684 0.34434555972075376 rpy=0 0 0 -> xyz=0 0.48820175054702664 0.8281490012226346 rpy=0 0 0
- joint Link3_Link4: origin xyz=0 0.8988646662309098 0.7396883322632737 rpy=0 0 0 -> xyz=0 0.233756348616039 0.07162717173401223 rpy=0 0 0
- joint Link4_Link5: origin xyz=0 0.6022585213627594 0.7539458440226775 rpy=0 0 0 -> xyz=0 0.7114452413300312 0.6620237559790881 rpy=0 0 0
- joint Link5_Link6: origin xyz=0 0.2471946032366631 0.697997747025809 rpy=0 0 0 -> xyz=0 0.4849924955659737 0.1457264134121834 rpy=0 0 0
- joint Link6_Link7: origin xyz=0 0.5166362385928098 0.4242463320739529 rpy=0 0 0 -> xyz=0 0.8234380003730708 0.953817394295689 rpy=0 0 0
- joint Link7_Link8: origin xyz=0 0.49852502806705734 0.895738399873903 rpy=0 0 0 -> xyz=0 0.76079497129132 0.186407095701565 rpy=0 0 0
- joint Link8_Link9: origin xyz=0 0.7256492995698836 0.5397813135865623 rpy=0 0 0 -> xyz=0 0.9055970329906969 0.8884605437782 rpy=0 0 0
- joint Link9_Link10: origin xyz=0 0.5927177378189967 0.21808294324593447 rpy=0 0 0 -> xyz=0 0.5195126159055607 0.38693715368187753 rpy=0 0 0

Commit message: some change

File: body.urdf (robot description, URDF)
Before this commit: robot robot, 10 links, 10 joints
Links:
- removed link Link0
- removed link Link8
- removed link Link9
- link Link1: geometry collision box size=0.4682901695840416 0.27062659899087393 0.2090453568031051; visual box size=0.4682901695840416 0.27062659899087393 0.2090453568031051
- link Link2: geometry collision box size=0.08721247073330168 0.3656675170523785 0.24721735750712293; visual box size=0.08721247073330168 0.3656675170523785 0.24721735750712293
- link Link3: geometry collision box size=0.34684514145931533 0.49694279854165363 0.2888836510083693; visual box size=0.34684514145931533 0.49694279854165363 0.2888836510083693
- link Link4: geometry collision box size=0.44235122609977867 0.02347741545590204 0.03677489851420873; visual box size=0.44235122609977867 0.02347741545590204 0.03677489851420873
- link Link5: geometry collision box size=0.45495060641337676 0.08429205276572238 0.13438958174545268; visual box size=0.45495060641337676 0.08429205276572238 0.13438958174545268
- link Link6: geometry collision box size=0.33232700615471883 0.3634364021846306 0.021717101098212455; visual box size=0.33232700615471883 0.3634364021846306 0.021717101098212455
- link Link7: geometry collision box size=0.45194275176850646 0.3249871939615555 0.3970840563831874; visual box size=0.45194275176850646 0.3249871939615555 0.3970840563831874
Joints:
- removed joint Link0_Link1
- removed joint Link7_Link8
- removed joint Link8_Link9
- removed joint Link9_Link10
- joint Link1_Link2: axis 1 0 0 -> 0 1 0; origin xyz=0 0.19415024083530874 0.936509516854282 rpy=0 0 0 -> xyz=0.2341450847920208 0 0.2090453568031051 rpy=0 0 0
- joint Link2_Link3: axis 1 0 0 -> 0 1 0; origin xyz=0 0.48820175054702664 0.8281490012226346 rpy=0 0 0 -> xyz=0.08721247073330168 0 0.24721735750712293 rpy=0 0 0
- joint Link3_Link4: axis 1 0 0 -> 0 1 0; origin xyz=0 0.233756348616039 0.07162717173401223 rpy=0 0 0 -> xyz=0.34684514145931533 0 0.2888836510083693 rpy=0 0 0
- joint Link4_Link5: axis 1 0 0 -> 0 1 0; origin xyz=0 0.7114452413300312 0.6620237559790881 rpy=0 0 0 -> xyz=0.44235122609977867 0 0.03677489851420873 rpy=0 0 0
- joint Link5_Link6: axis 1 0 0 -> 0 1 0; origin xyz=0 0.4849924955659737 0.1457264134121834 rpy=0 0 0 -> xyz=0.45495060641337676 0 0.13438958174545268 rpy=0 0 0
- joint Link6_Link7: axis 1 0 0 -> 0 1 0; origin xyz=0 0.8234380003730708 0.953817394295689 rpy=0 0 0 -> xyz=0.33232700615471883 0 0.021717101098212455 rpy=0 0 0

Commit message: 6 done

File: body.urdf (robot description, URDF)
Before this commit: robot robot, 7 links, 6 joints
Links:
- removed link Link5
- removed link Link6
- removed link Link7
- added link Link0, mass 1; collision box size=0.422115585827912 0.920845747988892 0.276108834875504; visual box size=0.422115585827912 0.920845747988892 0.276108834875504
- link Link1: geometry collision box size=0.8694046619033527 0.4955581657358684 0.07170467828039861; visual box size=0.8694046619033527 0.4955581657358684 0.07170467828039861
- link Link2: geometry collision box size=0.5606379114658376 0.1238595884644661 0.014438564279818267; visual box size=0.5606379114658376 0.1238595884644661 0.014438564279818267
- link Link3: geometry collision box size=0.1512264558107128 0.3359105872829752 0.5174816309082785; visual box size=0.1512264558107128 0.3359105872829752 0.5174816309082785
- link Link4: geometry collision box size=0.5812727893602095 0.6533348520515698 0.21527788706296114; visual box size=0.5812727893602095 0.6533348520515698 0.21527788706296114
Joints:
- removed joint Link4_Link5
- removed joint Link5_Link6
- removed joint Link6_Link7
- added joint Link0_Link1: type revolute, parent Link0, child Link1, origin xyz=0 0.460422873994446 0.276108834875504 rpy=0 0 0, axis 1 0 0, limit lower=-3.14159 upper=3.14159 effort=0.0 velocity=0.0
- joint Link1_Link2: axis 0 1 0 -> 1 0 0; origin xyz=0.2341450847920208 0 0.2090453568031051 rpy=0 0 0 -> xyz=0 0.4955581657358684 0.07170467828039861 rpy=0 0 0
- joint Link2_Link3: axis 0 1 0 -> 1 0 0; origin xyz=0.08721247073330168 0 0.24721735750712293 rpy=0 0 0 -> xyz=0 0.1238595884644661 0.014438564279818267 rpy=0 0 0
- joint Link3_Link4: axis 0 1 0 -> 1 0 0; origin xyz=0.34684514145931533 0 0.2888836510083693 rpy=0 0 0 -> xyz=0 0.3359105872829752 0.5174816309082785 rpy=0 0 0

Commit message: assign 7

File: body.urdf (robot description, URDF)
Before this commit: robot robot, 5 links, 4 joints
Links:
- added link Link5, mass 1; collision box size=0.37962591114429367 0.11188277302467675 0.6220835250091115; visual box size=0.37962591114429367 0.11188277302467675 0.6220835250091115
- added link Link6, mass 1; collision box size=0.9142239550870243 0.30767902790830814 0.31388937824139695; visual box size=0.9142239550870243 0.30767902790830814 0.31388937824139695
- added link Link7, mass 1; collision box size=0.5358033767269528 0.8002187192936902 0.6759823431928081; visual box size=0.5358033767269528 0.8002187192936902 0.6759823431928081
- added link Link8, mass 1; collision box size=0.23027041902786705 0.6129188201352119 0.9102563210741763; visual box size=0.23027041902786705 0.6129188201352119 0.9102563210741763
- added link Link9, mass 1; collision box size=0.6017040021076175 0.1885762663942826 0.10355726109610375; visual box size=0.6017040021076175 0.1885762663942826 0.10355726109610375
- link Link0: geometry collision box size=0.9795679306413696 0.20762386864234195 0.6743135074941482; visual box size=0.9795679306413696 0.20762386864234195 0.6743135074941482
- link Link1: geometry collision box size=0.9795679306413696 0.20762386864234195 0.6743135074941482; visual box size=0.9795679306413696 0.20762386864234195 0.6743135074941482
- link Link2: geometry collision box size=0.2995411965312611 0.8347413721635963 0.5715918446796506; visual box size=0.2995411965312611 0.8347413721635963 0.5715918446796506
- link Link3: geometry collision box size=0.004586178366824956 0.5137402288538597 0.43329894397301727; visual box size=0.004586178366824956 0.5137402288538597 0.43329894397301727
- link Link4: geometry collision box size=0.21251759640286483 0.34584282069911154 0.17652026288918798; visual box size=0.21251759640286483 0.34584282069911154 0.17652026288918798
Joints:
- added joint Link4_Link5: type revolute, parent Link4, child Link5, origin xyz=0.0 0 0.0 rpy=0 0 0, axis 0 1 0, limit lower=-3.14159 upper=3.14159 effort=0.0 velocity=0.0
- added joint Link5_Link6: type revolute, parent Link5, child Link6, origin xyz=0.37962591114429367 0 0.6220835250091115 rpy=0 0 0, axis 0 1 0, limit lower=-3.14159 upper=3.14159 effort=0.0 velocity=0.0
- added joint Link6_Link7: type revolute, parent Link6, child Link7, origin xyz=0.9142239550870243 0 0.0 rpy=0 0 0, axis 0 1 0, limit lower=-3.14159 upper=3.14159 effort=0.0 velocity=0.0
- added joint Link7_Link8: type revolute, parent Link7, child Link8, origin xyz=0.2679016883634764 0.4001093596468451 0.0 rpy=0 0 0, axis 1 0 0, limit lower=-3.14159 upper=3.14159 effort=0.0 velocity=0.0
- added joint Link8_Link9: type revolute, parent Link8, child Link9, origin xyz=-0.11513520951393352 0.30645941006760596 0.9102563210741763 rpy=0 0 0, axis 0 1 0, limit lower=-3.14159 upper=3.14159 effort=0.0 velocity=0.0
- joint Link0_Link1: origin xyz=0 0.460422873994446 0.276108834875504 rpy=0 0 0 -> xyz=0 0.10381193432117097 2.674313507494148 rpy=0 0 0
- joint Link1_Link2: axis 1 0 0 -> 0 1 0; origin xyz=0 0.4955581657358684 0.07170467828039861 rpy=0 0 0 -> xyz=-0.4897839653206848 0.10381193432117097 0.0 rpy=0 0 0
- joint Link2_Link3: axis 1 0 0 -> 0 1 0; origin xyz=0 0.1238595884644661 0.014438564279818267 rpy=0 0 0 -> xyz=-0.2995411965312611 0 0.0 rpy=0 0 0
- joint Link3_Link4: axis 1 0 0 -> 0 1 0; origin xyz=0 0.3359105872829752 0.5174816309082785 rpy=0 0 0 -> xyz=-0.004586178366824956 0 0.0 rpy=0 0 0
