Commit message: readme update

File: body.urdf (robot description, URDF)
Before this commit: robot robot, 10 links, 9 joints
Links:
- removed link Link6
- removed link Link7
- removed link Link8
- removed link Link9
- link Link0: geometry collision box size=0.22968587720172107 0.39345261923962993 0.2111227348890733; visual box size=0.22968587720172107 0.39345261923962993 0.2111227348890733
- link Link1: geometry collision box size=0.22968587720172107 0.39345261923962993 0.2111227348890733; visual box size=0.22968587720172107 0.39345261923962993 0.2111227348890733
- link Link2: geometry collision box size=0.7205213442898475 0.1252685442307392 0.6476298351873754; visual box size=0.7205213442898475 0.1252685442307392 0.6476298351873754
- link Link3: geometry collision box size=0.752730594281137 0.004671276814289693 0.07021699446988061; visual box size=0.752730594281137 0.004671276814289693 0.07021699446988061
- link Link4: geometry collision box size=0.35707981970789027 0.7200282236934472 0.31002951699555226; visual box size=0.35707981970789027 0.7200282236934472 0.31002951699555226
- link Link5: geometry collision box size=0.6236222432818485 0.7626366118592083 0.09767278899982668; visual box size=0.6236222432818485 0.7626366118592083 0.09767278899982668
Joints:
- removed joint Link5_Link6
- removed joint Link6_Link7
- removed joint Link7_Link8
- removed joint Link8_Link9
- joint Link0_Link1: origin xyz=0 0.10381193432117097 2.674313507494148 rpy=0 0 0 -> xyz=0 0.19672630961981497 2.211122734889073 rpy=0 0 0
- joint Link1_Link2: axis 0 1 0 -> 1 0 0; origin xyz=-0.4897839653206848 0.10381193432117097 0.0 rpy=0 0 0 -> xyz=0 0.39345261923962993 0.0 rpy=0 0 0
- joint Link2_Link3: origin xyz=-0.2995411965312611 0 0.0 rpy=0 0 0 -> xyz=0.36026067214492374 0.0626342721153696 0.6476298351873754 rpy=0 0 0
- joint Link3_Link4: origin xyz=-0.004586178366824956 0 0.0 rpy=0 0 0 -> xyz=0.752730594281137 0 0.0 rpy=0 0 0

Commit message: init changes

File: body.urdf (robot description, URDF)
Before this commit: robot robot, 6 links, 5 joints
Links:
- removed link Link4
- removed link Link5
- link Link0: geometry collision box size=0.6232848121231013 0.05169026617714667 0.6878271223593972; visual box size=0.6232848121231013 0.05169026617714667 0.6878271223593972
- link Link1: geometry collision box size=0.6232848121231013 0.05169026617714667 0.6878271223593972; visual box size=0.6232848121231013 0.05169026617714667 0.6878271223593972
- link Link2: geometry collision box size=0.4349939331757644 0.7793928720897072 0.9660090131755005; visual box size=0.4349939331757644 0.7793928720897072 0.9660090131755005
- link Link3: geometry collision box size=0.180100001911511 0.5077766675898346 0.3456890989982333; visual box size=0.180100001911511 0.5077766675898346 0.3456890989982333
Joints:
- removed joint Link3_Link4
- removed joint Link4_Link5
- joint Link0_Link1: origin xyz=0 0.19672630961981497 2.211122734889073 rpy=0 0 0 -> xyz=0 0.025845133088573335 2.6878271223593972 rpy=0 0 0
- joint Link1_Link2: axis 1 0 0 -> 0 1 0; origin xyz=0 0.39345261923962993 0.0 rpy=0 0 0 -> xyz=0.31164240606155064 0.025845133088573335 0.0 rpy=0 0 0
- joint Link2_Link3: origin xyz=0.36026067214492374 0.0626342721153696 0.6476298351873754 rpy=0 0 0 -> xyz=0.4349939331757644 0 0.9660090131755005 rpy=0 0 0
